Commit message: New robot description with melodic-devel-staging xacro. added a gazebo control plugin and a fixed link

File: homestri_robot/homestri_robot_description/urdf/ur5_e_robotiq_2f_85_macro.urdf.xacro (robot description, xacro)
@@ -1,32 +1,55 @@
 <?xml version="1.0"?>
-<robot xmlns:xacro="http://ros.org/wiki/xacro">
-  <!-- common stuff -->
-  <xacro:include filename="$(find ur_e_description)/urdf/common.gazebo.xacro" />
+<robot name="homestri_robot"
+  xmlns:xacro="http://ros.org/wiki/xacro">
   <!-- ur5e -->
-  <xacro:include filename="$(find ur_e_description)/urdf/ur5e.urdf.xacro" />
+  <!-- NOTE2: if you have a custom robot configuration, or your robot is
+  integrated into a work cell, do NOT change this file or add all of the
+  work cell objects to the ur.xacro file. Create a new top-level xacro and
+  include the ur_macro.xacro file into it. Then write a new .launch file
+  to load it onto the parameter server. -->
+  <xacro:include filename="$(find ur_description)/urdf/ur_macro.xacro"/>
+  <!-- parameters -->
+  <xacro:arg name="joint_limit_params" default="$(find ur_description)/config/ur5e/joint_limits.yaml"/>
+  <xacro:arg name="kinematics_params" default="$(find ur_description)/config/ur5e/default_kinematics.yaml"/>
+  <xacro:arg name="physical_params" default="$(find ur_description)/config/ur5e/physical_parameters.yaml"/>
+  <xacro:arg name="visual_params" default="$(find ur_description)/config/ur5e/visual_parameters.yaml"/>
+  <!-- legal values:
+         - hardware_interface/PositionJointInterface
+         - hardware_interface/VelocityJointInterface
+         - hardware_interface/EffortJointInterface
+   -->
+   <xacro:arg name="transmission_hw_interface" default="hardware_interface/PositionJointInterface"/>
+   <xacro:arg name="safety_limits" default="false"/>
+   <xacro:arg name="safety_pos_margin" default="0.15"/>
+   <xacro:arg name="safety_k_position" default="20"/>
   <!-- Gripper -->
-  <xacro:include filename="$(find robotiq_2f_85_gripper_visualization)/urdf/robotiq_arg2f_85_model_macro.xacro" />
+  <xacro:include filename="$(find robotiq_85_description)/urdf/robotiq_85_gripper.urdf.xacro" />
+  <!-- instantiate everything -->
   <xacro:macro name="ur5_e_robotiq_2f_85" params="prefix">
-    <!-- This is where joint limits should be made -->
-    <xacro:ur5e_robot prefix="${prefix}" joint_limited="true"
-      shoulder_pan_lower_limit="${-pi}" shoulder_pan_upper_limit="${pi}"
-      shoulder_lift_lower_limit="${-pi}" shoulder_lift_upper_limit="${pi}"
-      elbow_joint_lower_limit="${-pi}" elbow_joint_upper_limit="${pi}"
-      wrist_1_lower_limit="${-pi}" wrist_1_upper_limit="${pi}"
-      wrist_2_lower_limit="${-pi}" wrist_2_upper_limit="${pi}"
-      wrist_3_lower_limit="${-pi}" wrist_3_upper_limit="${pi}"
-    />
-    <xacro:robotiq_arg2f_85 prefix="${prefix}" />
-      <link name="world"/>
-      <joint name="world-base" type="fixed">
-        <origin xyz="0 0 0" rpy="0 0 0" />
-        <parent link="world" />
-        <child link="${prefix}base_link" />
-      </joint>
-      <joint name="connector" type="fixed">
-        <origin xyz="0 0 0" rpy="0 ${pi / 2} 0" />
-        <parent link="${prefix}ee_link" />
-        <child link="${prefix}robotiq_arg2f_base_link" />
-      </joint>
+   <!-- arm -->
+   <xacro:ur_robot
+     prefix="${prefix}"
+     joint_limits_parameters_file="$(arg joint_limit_params)"
+     kinematics_parameters_file="$(arg kinematics_params)"
+     physical_parameters_file="$(arg physical_params)"
+     visual_parameters_file="$(arg visual_params)"
+     transmission_hw_interface="$(arg transmission_hw_interface)"
+     safety_limits="$(arg safety_limits)"
+     safety_pos_margin="$(arg safety_pos_margin)"
+     safety_k_position="$(arg safety_k_position)"/>
+    <xacro:robotiq_85_gripper prefix="${prefix}" parent="${prefix}flange">
+      <origin xyz="0 0 0" rpy="0 0 0"/>
+    </xacro:robotiq_85_gripper>
+    <link name="world"/>
+    <joint name="world-base" type="fixed">
+      <origin xyz="0 0 0" rpy="0 0 0" />
+      <parent link="world" />
+      <child link="${prefix}base_link" />
+    </joint>
+    <!-- Use this for gazebo, omit gazebo for real robot -->
+    <gazebo>
+      <plugin name="gazebo_ros_control" filename="libgazebo_ros_control.so">
+      </plugin>
+    </gazebo>
   </xacro:macro>
 </robot>
