Commit message: new interface for position spawning

File: homestri_robot/homestri_robot_description/urdf/ur5_e_robotiq_2f_85.urdf.xacro (robot description, xacro)
@@ -1,5 +1,7 @@
 <?xml version="1.0"?>
 <robot name="robot_arm" xmlns:xacro="http://ros.org/wiki/xacro">
+  <xacro:arg name="xyz" default="0 0 0" />
+  <xacro:arg name="rpy" default="0 0 0" />
   <xacro:include filename="$(find homestri_robot_description)/urdf/ur5_e_robotiq_2f_85_macro.urdf.xacro" />
-  <xacro:ur5_e_robotiq_2f_85 prefix=""/>
+  <xacro:ur5_e_robotiq_2f_85 prefix="" origin_xyz="$(arg xyz)" origin_rpy="$(arg rpy)"/>
 </robot>

File: homestri_robot/homestri_robot_description/urdf/ur5_e_robotiq_2f_85_macro.urdf.xacro (robot description, xacro)
@@ -26,5 +26,5 @@
   <xacro:include filename="$(find robotiq_85_description)/urdf/robotiq_85_gripper.urdf.xacro" />
   <!-- instantiate everything -->
-  <xacro:macro name="ur5_e_robotiq_2f_85" params="prefix">
+  <xacro:macro name="ur5_e_robotiq_2f_85" params="prefix origin_xyz origin_rpy">
    <!-- arm -->
    <xacro:ur_robot
@@ -43,5 +43,5 @@
     <link name="world"/>
     <joint name="world-base" type="fixed">
-      <origin xyz="0 0 0" rpy="0 0 0" />
+      <origin xyz="${origin_xyz}" rpy="${origin_rpy}" />
       <parent link="world" />
       <child link="${prefix}base_link" />
